File: kicad/3ric/mono_qvga.kicad_sch (KiCad schematic)
At the start: 5 parts

Commit message: schematic updates - bring the schematics up to match breadboard changes current state has high res Apple II color emulation working
Parts:
- removed J_VGA1: DB15_Female_HighDensity, Connector_Dsub:DSUB-15-HD_Female_Horizontal_P2.29x1.98mm_EdgePinOffset8.35mm_Housed_MountingHolesOffset10.89mm, symbol Connector:DB15_Female_HighDensity
- removed U_AND_OUT1: 74LS08, Package_DIP:DIP-14_W7.62mm_Socket, symbol 74xx:74LS08
- removed U_CLOCK_DIV1: 74LS161, Package_DIP:DIP-16_W7.62mm_Socket, symbol 74xx:74LS161
- removed U_XOR1: 74LS86, Package_DIP:DIP-14_W7.62mm_Socket, symbol 74xx:74LS86
- removed X_CLK_VGA1: 25.175MHz, Oscillator:Oscillator_DIP-14, symbol Oscillator:ACO-xxxMHz
Connections:
- no-connect marks 18 -> 0
Other:
- removed sheet caps
- removed sheet textmode
- removed sheet vga_memsignal
- removed sheet vga_vidmem
- removed sheet vgatiming
