File: kicad/3ric/serial.kicad_sch (KiCad schematic)
At the start: 3 parts, among them J2 Conn_02x03_Odd_Even, U10 6502-library_65C51N

Commit message: schematic updates - bring the schematics up to match breadboard changes current state has high res Apple II color emulation working
Parts:
- removed J2: Conn_02x03_Odd_Even, Connector_PinHeader_2.54mm:PinHeader_2x03_P2.54mm_Vertical, symbol Connector_Generic:Conn_02x03_Odd_Even
- removed U10: 6502-library_65C51N, Package_DIP:DIP-28_W15.24mm_Socket, symbol EB6502-custom:6502-library_65C51N
- removed X_CLK_ACIA1: 1.8432MHz, Oscillator:Oscillator_DIP-14, symbol Oscillator:ACO-xxxMHz
Connections:
- no-connect marks 4 -> 0
