File: kicad/3ric/vga_vidmem.kicad_sch (KiCad schematic)
At the start: 10 parts

Commit message: cleaning up of the schematic
Parts:
- removed C2_NOT, U? (x2): 74LS04, symbol 74xx:74LS04
- added unit 6 of N7_NOT1
- added unit 5 of N7_NOT1
- N7_NOT1: renamed from N7_NOT; footprint (none) -> Package_DIP:DIP-14_W7.62mm_Socket
- renumbered N3_ADDR_CNT to N3_ADDR_CNT1, N4_ADDR_CNT to N4_ADDR_CNT1, N5_ADDR_CNT to N5_ADDR_CNT1, N6_ADDR_CNT to N6_ADDR_CNT1, O2_ROM_VADDR_LOW to O2_ROM_VADDR_LOW1, O3_ROM_VADDR_HIGH to O3_ROM_VADDR_HIGH1
Connections:
- net !Display2 renamed !DISPLAY2
- net Display2 renamed DISPLAY2
- new net CA7: N7_NOT1.11
- new net ~{CA7}: N7_NOT1.10
- no-connect marks 1 -> 3

Commit message: pcb layout continued
Connections:
- net !DISPLAY2 is gone; now on net ~{CA7}: N7_NOT1.8
- net DISPLAY2 is gone; now on net CA7: N7_NOT1.9
- net !GFXSHIFT: now also N7_NOT1.12; no longer N7_NOT1.4
- net !LOWSHIFT: now also N7_NOT1.10; no longer N7_NOT1.6
- net CA7: no longer N7_NOT1.11
- net GFXSHIFT: now also N7_NOT1.13; no longer N7_NOT1.3
- net LOWSHIFT: now also N7_NOT1.11; no longer N7_NOT1.5
- net ~{CA7}: no longer N7_NOT1.10
- net FULLMODE renamed MIXEDMODE
- net GFXMODE renamed TEXTMODE
- net PAGE1 renamed PAGE2
- no-connect marks 3 -> 5
Other:
- moved on the sheet: N7_NOT1F
