File: kicad/3ric/3ric.kicad_pcb (KiCad board)
At the start: 4 copper layers, 0 parts

Commit message: updated schematics and PCB PNG of the breadboard layout
Parts:
- added A1: 74LS08, Package_DIP:DIP-14_W7.62mm_Socket, F.Cu at (52.8, 134.7)
- added A2: 74LS32, Package_DIP:DIP-14_W7.62mm_Socket, F.Cu at (67.5, 134.7)
- added A3: 74LS08, Package_DIP:DIP-14_W7.62mm_Socket, F.Cu at (83.2, 134.9)
- added A4: 74LS32, Package_DIP:DIP-14_W7.62mm_Socket, F.Cu at (99.0, 135.0)
- added A5: 74LS08, Package_DIP:DIP-14_W7.62mm_Socket, F.Cu at (114.5, 135.0)
- added B1: 74LS08, Package_DIP:DIP-14_W7.62mm_Socket, F.Cu at (37.2, 134.7)
- added B2: 74LS00, Package_DIP:DIP-14_W7.62mm_Socket, F.Cu at (29.2, 159.4)
- added B3: 74LS32, Package_DIP:DIP-14_W7.62mm_Socket, F.Cu at (44.2, 159.4)
- added B4: 74LS32, Package_DIP:DIP-14_W7.62mm_Socket, F.Cu at (59.1, 159.3)
- added B5: 74LS08, Package_DIP:DIP-14_W7.62mm_Socket, F.Cu at (75.1, 159.3)
- added B6: 74LS04, Package_DIP:DIP-14_W7.62mm_Socket, F.Cu at (90.9, 159.0)
- added B7: 74LS00, Package_DIP:DIP-14_W7.62mm_Socket, F.Cu at (106.6, 159.0)
- added C1: 74LS32, Package_DIP:DIP-14_W7.62mm_Socket, F.Cu at (90.7, 197.9)
- added C10: 0.1µ, Capacitor_SMD:C_1206_3216Metric_Pad1.33x1.80mm_HandSolder, B.Cu at (279.6, 219.3)
- added C100: 0.1µ, Capacitor_SMD:C_1206_3216Metric_Pad1.33x1.80mm_HandSolder, B.Cu at (179.0, 126.0)
- added C101: 0.1µ, Capacitor_SMD:C_1206_3216Metric_Pad1.33x1.80mm_HandSolder, B.Cu at (177.7, 103.3)
- added C102: 0.1µ, Capacitor_SMD:C_1206_3216Metric_Pad1.33x1.80mm_HandSolder, B.Cu at (184.9, 80.9)
- added C103: 0.1µ, Capacitor_SMD:C_1206_3216Metric_Pad1.33x1.80mm_HandSolder, B.Cu at (80.2, 68.2)
- added C104: 0.1µ, Capacitor_SMD:C_1206_3216Metric_Pad1.33x1.80mm_HandSolder, B.Cu at (138.3, 69.4)
- added C105: 0.1µ, Capacitor_SMD:C_1206_3216Metric_Pad1.33x1.80mm_HandSolder, B.Cu at (151.3, 65.1)
- added C11: 0.1µ, Capacitor_SMD:C_1206_3216Metric_Pad1.33x1.80mm_HandSolder, B.Cu at (316.2, 134.9)
- added C12: 0.1µF, Capacitor_SMD:C_1206_3216Metric_Pad1.33x1.80mm_HandSolder, B.Cu at (257.7, 132.3)
- added C13: 0.1µ, Capacitor_SMD:C_1206_3216Metric_Pad1.33x1.80mm_HandSolder, B.Cu at (136.1, 266.9)
- added C14: 0.1µF, Capacitor_SMD:C_1206_3216Metric_Pad1.33x1.80mm_HandSolder, B.Cu at (121.8, 266.9)
- added C15: 0.1µ, Capacitor_SMD:C_1206_3216Metric_Pad1.33x1.80mm_HandSolder, B.Cu at (109.1, 267.5)
- added C16: 0.1µF, Capacitor_SMD:C_1206_3216Metric_Pad1.33x1.80mm_HandSolder, B.Cu at (95.2, 266.2)
- added C17: 0.1µF, Capacitor_SMD:C_1206_3216Metric_Pad1.33x1.80mm_HandSolder, B.Cu at (183.2, 231.1)
- added C18: 0.1µF, Capacitor_SMD:C_1206_3216Metric_Pad1.33x1.80mm_HandSolder, B.Cu at (183.2, 243.6)
- added C19: 0.1µF, Capacitor_SMD:C_1206_3216Metric_Pad1.33x1.80mm_HandSolder, B.Cu at (183.1, 256.3)
- added C2: 74LS04, Package_DIP:DIP-14_W7.62mm_Socket, F.Cu at (75.1, 197.8)
- added C20: 0.1µF, Capacitor_SMD:C_1206_3216Metric_Pad1.33x1.80mm_HandSolder, B.Cu at (157.3, 255.7)
- added C21: 0.1µF, Capacitor_SMD:C_1206_3216Metric_Pad1.33x1.80mm_HandSolder, B.Cu at (158.1, 271.5)
- added C22: 0.1µF, Capacitor_SMD:C_1206_3216Metric_Pad1.33x1.80mm_HandSolder, B.Cu at (79.6, 266.0)
- added C23: 0.1µF, Capacitor_SMD:C_1206_3216Metric_Pad1.33x1.80mm_HandSolder, B.Cu at (63.0, 265.0)
- added C24: 0.1µF, Capacitor_SMD:C_1206_3216Metric_Pad1.33x1.80mm_HandSolder, B.Cu at (47.5, 265.5)
- added C25: 0.1µF, Capacitor_SMD:C_1206_3216Metric_Pad1.33x1.80mm_HandSolder, B.Cu at (47.7, 238.0)
- added C26: 0.1µF, Capacitor_SMD:C_1206_3216Metric_Pad1.33x1.80mm_HandSolder, B.Cu at (63.4, 237.8)
- added C27: 0.1µF, Capacitor_SMD:C_1206_3216Metric_Pad1.33x1.80mm_HandSolder, B.Cu at (79.8, 239.1)
- added C28: 0.1µF, Capacitor_SMD:C_1206_3216Metric_Pad1.33x1.80mm_HandSolder, B.Cu at (95.6, 238.2)
- added C29: 0.1µF, Capacitor_SMD:C_1206_3216Metric_Pad1.33x1.80mm_HandSolder, B.Cu at (111.5, 238.7)
- added C3: C30, Capacitor_SMD:C_0805_2012Metric_Pad1.18x1.45mm_HandSolder, B.Cu at (296.4, 170.6)
- added C30: 0.1µF, Capacitor_SMD:C_1206_3216Metric_Pad1.33x1.80mm_HandSolder, B.Cu at (127.6, 238.4)
- added C31: 0.1µF, Capacitor_SMD:C_1206_3216Metric_Pad1.33x1.80mm_HandSolder, B.Cu at (152.3, 237.3)
- added C32: 0.1µF, Capacitor_SMD:C_1206_3216Metric_Pad1.33x1.80mm_HandSolder, B.Cu at (56.1, 215.2)
- added C33: 0.1µF, Capacitor_SMD:C_1206_3216Metric_Pad1.33x1.80mm_HandSolder, B.Cu at (71.3, 214.4)
- added C34: 0.1µF, Capacitor_SMD:C_1206_3216Metric_Pad1.33x1.80mm_HandSolder, B.Cu at (87.0, 214.3)
- added C35: 0.1µF, Capacitor_SMD:C_1206_3216Metric_Pad1.33x1.80mm_HandSolder, B.Cu at (40.7, 190.5)
- added C36: 0.1µF, Capacitor_SMD:C_1206_3216Metric_Pad1.33x1.80mm_HandSolder, B.Cu at (114.4, 214.4)
- added C37: 0.1µF, Capacitor_SMD:C_1206_3216Metric_Pad1.33x1.80mm_HandSolder, B.Cu at (113.8, 191.7)
- added C38: 0.1µF, Capacitor_SMD:C_1206_3216Metric_Pad1.33x1.80mm_HandSolder, B.Cu at (146.8, 211.4)
- added C39: 0.1µF, Capacitor_SMD:C_1206_3216Metric_Pad1.33x1.80mm_HandSolder, B.Cu at (282.5, 256.6)
- added C4: C106, Capacitor_SMD:C_0603_1608Metric_Pad1.08x0.95mm_HandSolder, B.Cu at (308.5, 181.0)
- added C40: 0.1µF, Capacitor_SMD:C_1206_3216Metric_Pad1.33x1.80mm_HandSolder, B.Cu at (192.4, 275.4)
- added C41: 0.1µF, Capacitor_SMD:C_1206_3216Metric_Pad1.33x1.80mm_HandSolder, B.Cu at (228.3, 242.7)
- added C42: 0.1µF, Capacitor_SMD:C_1206_3216Metric_Pad1.33x1.80mm_HandSolder, B.Cu at (205.3, 242.4)
- added C43: 0.1µF, Capacitor_SMD:C_1206_3216Metric_Pad1.33x1.80mm_HandSolder, B.Cu at (230.8, 276.0)
- added C44: 0.1µF, Capacitor_SMD:C_1206_3216Metric_Pad1.33x1.80mm_HandSolder, B.Cu at (156.9, 159.1)
- added C45: 0.1µF, Capacitor_SMD:C_1206_3216Metric_Pad1.33x1.80mm_HandSolder, B.Cu at (139.5, 188.6)
- added C46: 0.1µF, Capacitor_SMD:C_1206_3216Metric_Pad1.33x1.80mm_HandSolder, B.Cu at (186.8, 206.3)
- added C47: 0.1µF, Capacitor_SMD:C_1206_3216Metric_Pad1.33x1.80mm_HandSolder, B.Cu at (201.7, 207.4)
- added C48: 106, Capacitor_SMD:C_0603_1608Metric_Pad1.08x0.95mm_HandSolder, B.Cu at (307.5, 77.4)
- added C49: 106, Capacitor_SMD:C_0603_1608Metric_Pad1.08x0.95mm_HandSolder, B.Cu at (311.5, 69.6)
- added C5: 74LS08, Package_DIP:DIP-14_W7.62mm_Socket, F.Cu at (59.2, 198.0)
- added C50: 106, Capacitor_SMD:C_0603_1608Metric_Pad1.08x0.95mm_HandSolder, B.Cu at (315.3, 77.2)
- added C51: 106, Capacitor_SMD:C_0603_1608Metric_Pad1.08x0.95mm_HandSolder, B.Cu at (318.6, 69.5)
- added C52: 0.1µF, Capacitor_SMD:C_1206_3216Metric_Pad1.33x1.80mm_HandSolder, B.Cu at (110.5, 166.7)
- added C53: 0.1µF, Capacitor_SMD:C_1206_3216Metric_Pad1.33x1.80mm_HandSolder, B.Cu at (201.4, 179.0)
- added C54: 0.1µF, Capacitor_SMD:C_1206_3216Metric_Pad1.33x1.80mm_HandSolder, B.Cu at (174.4, 152.1)
- added C55: 0.1µF, Capacitor_SMD:C_1206_3216Metric_Pad1.33x1.80mm_HandSolder, B.Cu at (217.1, 162.7)
- added C56: 0.1µF, Capacitor_SMD:C_1206_3216Metric_Pad1.33x1.80mm_HandSolder, B.Cu at (217.8, 188.8)
- added C57: 0.1µ, Capacitor_SMD:C_1206_3216Metric_Pad1.33x1.80mm_HandSolder, B.Cu at (201.3, 150.2)
- added C59: 0.1µF, Capacitor_SMD:C_1206_3216Metric_Pad1.33x1.80mm_HandSolder, B.Cu at (231.3, 167.1)
- added C6: 0.1µ, Capacitor_SMD:C_1206_3216Metric_Pad1.33x1.80mm_HandSolder, B.Cu at (281.9, 279.0)
- added C60: 0.1µF, Capacitor_SMD:C_1206_3216Metric_Pad1.33x1.80mm_HandSolder, B.Cu at (234.6, 201.6)
- added C61: 0.1µF, Capacitor_SMD:C_1206_3216Metric_Pad1.33x1.80mm_HandSolder, B.Cu at (94.7, 166.9)
- added C62: 0.1µF, Capacitor_SMD:C_1206_3216Metric_Pad1.33x1.80mm_HandSolder, B.Cu at (187.8, 167.4)
- added C63: 0.1µ, Capacitor_SMD:C_1206_3216Metric_Pad1.33x1.80mm_HandSolder, B.Cu at (293.4, 108.3)
- added C64: 0.1µF, Capacitor_SMD:C_1206_3216Metric_Pad1.33x1.80mm_HandSolder, B.Cu at (322.6, 108.1)
- added C65: 0.1µF, Capacitor_SMD:C_1206_3216Metric_Pad1.33x1.80mm_HandSolder, B.Cu at (308.1, 108.2)
- added C66: 0.1µF, Capacitor_SMD:C_1206_3216Metric_Pad1.33x1.80mm_HandSolder, B.Cu at (322.1, 166.8)
- added C67: 0.1µF, Capacitor_SMD:C_1206_3216Metric_Pad1.33x1.80mm_HandSolder, B.Cu at (309.7, 166.1)
- added C68: 0.1µ, Capacitor_SMD:C_1206_3216Metric_Pad1.33x1.80mm_HandSolder, B.Cu at (296.3, 159.5)
- added C69: 0.1µF, Capacitor_SMD:C_1206_3216Metric_Pad1.33x1.80mm_HandSolder, B.Cu at (279.5, 108.2)
- added C7: 0.1µF, Capacitor_SMD:C_1206_3216Metric_Pad1.33x1.80mm_HandSolder, B.Cu at (264.2, 165.2)
- added C70: 0.1µF, Capacitor_SMD:C_1206_3216Metric_Pad1.33x1.80mm_HandSolder, B.Cu at (118.3, 142.5)
- added C71: 0.1µF, Capacitor_SMD:C_1206_3216Metric_Pad1.33x1.80mm_HandSolder, B.Cu at (62.9, 166.8)
- added C72: 0.1µF, Capacitor_SMD:C_1206_3216Metric_Pad1.33x1.80mm_HandSolder, B.Cu at (79.0, 166.8)
- added C73: 0.1µ, Capacitor_SMD:C_1206_3216Metric_Pad1.33x1.80mm_HandSolder, B.Cu at (221.3, 108.4)
- added C74: 0.1µ, Capacitor_SMD:C_1206_3216Metric_Pad1.33x1.80mm_HandSolder, B.Cu at (235.7, 108.4)
- added C75: 0.1µ, Capacitor_SMD:C_1206_3216Metric_Pad1.33x1.80mm_HandSolder, B.Cu at (243.2, 135.0)
- added C76: 0.1µ, Capacitor_SMD:C_1206_3216Metric_Pad1.33x1.80mm_HandSolder, B.Cu at (250.8, 108.4)
- added C77: 0.1µ, Capacitor_SMD:C_1206_3216Metric_Pad1.33x1.80mm_HandSolder, B.Cu at (265.1, 108.3)
- added C78: 0.1µ, Capacitor_SMD:C_1206_3216Metric_Pad1.33x1.80mm_HandSolder, B.Cu at (300.4, 134.1)
- added C79: 0.1µ, Capacitor_SMD:C_1206_3216Metric_Pad1.33x1.80mm_HandSolder, B.Cu at (56.7, 142.4)
- added C8: 0.1µ, Capacitor_SMD:C_1206_3216Metric_Pad1.33x1.80mm_HandSolder, B.Cu at (272.2, 131.4)
- added C80: 0.1µ, Capacitor_SMD:C_1206_3216Metric_Pad1.33x1.80mm_HandSolder, B.Cu at (71.4, 142.5)
- added C81: 0.1µ, Capacitor_SMD:C_1206_3216Metric_Pad1.33x1.80mm_HandSolder, B.Cu at (33.1, 166.8)
- added C82: 0.1µ, Capacitor_SMD:C_1206_3216Metric_Pad1.33x1.80mm_HandSolder, B.Cu at (48.1, 167.0)
- added C83: 0.1µ, Capacitor_SMD:C_1206_3216Metric_Pad1.33x1.80mm_HandSolder, B.Cu at (87.0, 142.8)
- added C85: 0.1µ, Capacitor_SMD:C_1206_3216Metric_Pad1.33x1.80mm_HandSolder, B.Cu at (102.7, 142.6)
- added C86: 0.1µ, Capacitor_SMD:C_1206_3216Metric_Pad1.33x1.80mm_HandSolder, B.Cu at (286.4, 134.4)
- added C87: 0.1µ, Capacitor_SMD:C_1206_3216Metric_Pad1.33x1.80mm_HandSolder, B.Cu at (136.2, 154.2)
- added C88: 0.1µ, Capacitor_SMD:C_1206_3216Metric_Pad1.33x1.80mm_HandSolder, B.Cu at (86.9, 190.9)
- added C89: 0.1µ, Capacitor_SMD:C_1206_3216Metric_Pad1.33x1.80mm_HandSolder, B.Cu at (71.2, 190.4)
- added C9: 0.1µF, Capacitor_SMD:C_1206_3216Metric_Pad1.33x1.80mm_HandSolder, B.Cu at (279.9, 197.2)
- added C90: 0.1µ, Capacitor_SMD:C_1206_3216Metric_Pad1.33x1.80mm_HandSolder, B.Cu at (55.3, 190.5)
- added C95: 0.1µ, Capacitor_SMD:C_1206_3216Metric_Pad1.33x1.80mm_HandSolder, B.Cu at (41.0, 142.4)
- added C96: 0.1µ, Capacitor_SMD:C_1206_3216Metric_Pad1.33x1.80mm_HandSolder, B.Cu at (174.6, 183.8)
- added C97: 0.1µ, Capacitor_SMD:C_1206_3216Metric_Pad1.33x1.80mm_HandSolder, B.Cu at (228.7, 134.9)
- added C98: 0.1µ, Capacitor_SMD:C_1206_3216Metric_Pad1.33x1.80mm_HandSolder, B.Cu at (216.5, 136.3)
- added C99: 0.1µ, Capacitor_SMD:C_1206_3216Metric_Pad1.33x1.80mm_HandSolder, B.Cu at (145.4, 94.1)
- added C_RESET_1: 0.1µF, Capacitor_SMD:C_1206_3216Metric_Pad1.33x1.80mm_HandSolder, B.Cu at (41.4, 125.2)
- added D1: 74LS32, Package_DIP:DIP-14_W7.62mm_Socket, F.Cu at (51.8, 206.4)
- added D10: D, Diode_SMD:D_SMA-SMB_Universal_Handsoldering, B.Cu at (314.3, 250.9)
- added D11: D, Diode_SMD:D_SMA-SMB_Universal_Handsoldering, B.Cu at (314.1, 257.2)
- added D12: D, Diode_SMD:D_SMA-SMB_Universal_Handsoldering, B.Cu at (314.4, 263.2)
- added D2: 74LS32, Package_DIP:DIP-14_W7.62mm_Socket, F.Cu at (67.6, 206.3)
- added D20: D, Diode_SMD:D_SMA-SMB_Universal_Handsoldering, B.Cu at (274.1, 88.3)
- added D21: D, Diode_SMD:D_SMA-SMB_Universal_Handsoldering, B.Cu at (265.1, 88.3)
- added D22: D, Diode_SMD:D_SMA-SMB_Universal_Handsoldering, B.Cu at (282.6, 88.3)
- added D23: D, Diode_SMD:D_SMA-SMB_Universal_Handsoldering, B.Cu at (290.6, 88.3)
- added D24: D, Diode_SMD:D_SMA-SMB_Universal_Handsoldering, B.Cu at (256.1, 88.3)
- added D3: 74LS32, Package_DIP:DIP-14_W7.62mm_Socket, F.Cu at (83.1, 206.2)
- added D4: 74LS00, Package_DIP:DIP-14_W7.62mm_Socket, F.Cu at (44.5, 198.2)
- added D5: 74LS154, Package_DIP:DIP-24_W15.24mm_Socket, F.Cu at (99.7, 221.6)
- added D6: 74LS154, Package_DIP:DIP-24_W15.24mm_Socket, F.Cu at (100.0, 199.2)
- added D7: D, Diode_SMD:D_SMA-SMB_Universal_Handsoldering, B.Cu at (313.4, 192.1)
- added D8: D, Diode_SMD:D_SMA-SMB_Universal_Handsoldering, B.Cu at (313.5, 198.3)
- added D9: D, Diode_SMD:D_SMA-SMB_Universal_Handsoldering, B.Cu at (313.6, 205.1)
- added E1: 74LS32, Package_DIP:DIP-14_W7.62mm_Socket, F.Cu at (43.9, 230.4)
- added E2: 74LS08, Package_DIP:DIP-14_W7.62mm_Socket, F.Cu at (59.3, 230.1)
- added E3: 74LS00, Package_DIP:DIP-14_W7.62mm_Socket, F.Cu at (75.8, 231.4)
- added E4: 74LS32, Package_DIP:DIP-14_W7.62mm_Socket, F.Cu at (91.6, 230.7)
- added E5: 74LS32, Package_DIP:DIP-14_W7.62mm_Socket, F.Cu at (108.0, 230.6)
- added E6: 74LS00, Package_DIP:DIP-14_W7.62mm_Socket, F.Cu at (123.6, 230.8)
- added F1: 74LS00, Package_DIP:DIP-14_W7.62mm_Socket, F.Cu at (43.7, 257.4)
- added F2: 74LS32, Package_DIP:DIP-14_W7.62mm_Socket, F.Cu at (59.0, 257.3)
- added F3: 74LS112, Package_DIP:DIP-16_W7.62mm_Socket, F.Cu at (75.4, 256.4)
- added F4: 74LS112, Package_DIP:DIP-16_W7.62mm_Socket, F.Cu at (91.3, 257.0)
- added F5: 74LS14, Package_DIP:DIP-14_W7.62mm_Socket, F.Cu at (105.0, 259.4)
- added F6: 74LS00, Package_DIP:DIP-14_W7.62mm_Socket, F.Cu at (118.0, 259.1)
- added F7: 74LS08, Package_DIP:DIP-14_W7.62mm_Socket, F.Cu at (132.0, 259.1)
- added H1: MountingHole, MountingHole:MountingHole_4.3mm_M4, F.Cu at (41.7, 59.4)
- added H10: MountingHole, MountingHole:MountingHole_4.3mm_M4, F.Cu at (323.6, 82.0)
- added H1_LEVEL_SHIFT1: ~, Package_SO:ETSSOP-20-1EP_4.4x6.5mm_P0.65mm_EP3x4.2mm, F.Cu at (196.8, 63.1)
- added H2: MountingHole, MountingHole:MountingHole_4.3mm_M4, F.Cu at (120.5, 59.4)
- added H2_ACIA_CLK1: 1.8432MHz, Oscillator:Oscillator_DIP-14, F.Cu at (138.3, 97.8)
- added H3: MountingHole, MountingHole:MountingHole_4.3mm_M4, F.Cu at (166.2, 59.4)
- added H4: MountingHole, MountingHole:MountingHole_4.3mm_M4, F.Cu at (166.2, 214.2)
- added H5: MountingHole, MountingHole:MountingHole_4.3mm_M4, F.Cu at (41.5, 214.1)
- added H6: MountingHole, MountingHole:MountingHole_4.3mm_M4, F.Cu at (166.2, 286.6)
- added H7: MountingHole, MountingHole:MountingHole_4.3mm_M4, F.Cu at (41.6, 286.6)
- added H8: MountingHole, MountingHole:MountingHole_4.3mm_M4, F.Cu at (323.6, 286.6)
- added H9: MountingHole, MountingHole:MountingHole_4.3mm_M4, F.Cu at (323.6, 214.2)
- added I1_VIA1: 65C22S, Package_DIP:DIP-40_W15.24mm_Socket, F.Cu at (208.8, 73.1)
- added J1: Conn_01x08, Connector_PinHeader_2.54mm:PinHeader_1x08_P2.54mm_Vertical, F.Cu at (298.3, 236.8)
- added J1_AND1: 74LS08, Package_DIP:DIP-14_W7.62mm_Socket, F.Cu at (200.8, 94.6)
- added J2: Conn_02x03_Odd_Even, Connector_PinHeader_2.54mm:PinHeader_2x03_P2.54mm_Vertical, F.Cu at (155.8, 188.2)
- added J3: STX-4235-3_3-N, audiojack:STX423533N, F.Cu at (311.8, 56.2)
- added J3_DEV_DECODE1: 74LS154, Package_DIP:DIP-24_W15.24mm_Socket, F.Cu at (128.2, 140.5)
- added J4: Conn_01x08, Connector_PinHeader_2.54mm:PinHeader_1x08_P2.54mm_Vertical, F.Cu at (272.2, 236.7)
- added J4_ACIA1: 6502-library_65C51N, Package_DIP:DIP-28_W15.24mm_Socket, F.Cu at (161.4, 110.5)
- added J5: Conn_02x08_Odd_Even, Connector_PinHeader_2.54mm:PinHeader_2x08_P2.54mm_Vertical, F.Cu at (154.2, 106.8)
- added J6: Conn_02x08_Odd_Even, Connector_PinHeader_2.54mm:PinHeader_2x08_P2.54mm_Vertical, F.Cu at (145.9, 129.0)
- added J_BEEP1: Conn_01x02_Pin, Connector_PinHeader_2.54mm:PinHeader_2x01_P2.54mm_Vertical, F.Cu at (30.4, 260.5)
- added J_POWER_1: Conn_01x02_Pin, Connector_PinHeader_2.54mm:PinHeader_2x01_P2.54mm_Vertical, F.Cu at (49.6, 124.3)
- added J_POWER_2: Conn_01x02_Pin, Connector_PinHeader_2.54mm:PinHeader_2x01_P2.54mm_Vertical, F.Cu at (30.9, 125.6)
- added J_POWER_3: ATX-24, atxplug:1-1775099-3, F.Cu at (87.1, 126.9)
- added J_RESET_1: Conn_01x02_Pin, Connector_PinHeader_2.54mm:PinHeader_2x01_P2.54mm_Vertical, F.Cu at (31.1, 117.8)
- added K1_CPU1: 6502-library_65C02S-2, Package_DIP:DIP-40_W15.24mm_Socket, F.Cu at (203.5, 118.2)
- added K2_ROM1: SST39SF040, Package_DIP:DIP-32_W15.24mm_Socket, F.Cu at (164.7, 177.8)
- added L1_RAM1: EB6502_isc61c1024-15n, Package_DIP:DIP-32_W7.62mm, F.Cu at (191.6, 185.6)
- added L2_BUS_A_LOW1: 74LS245, Package_DIP:DIP-20_W7.62mm_Socket, F.Cu at (170.8, 171.2)
- added L3_BUS_A_HIGH1: 74LS245, Package_DIP:DIP-20_W7.62mm_Socket, F.Cu at (170.5, 140.5)
- added L4_BUS_DATA1: 74LS245, Package_DIP:DIP-20_W7.62mm_Socket, F.Cu at (212.6, 124.3)
- added L5_VDATA_LATCH1: 74LS574, Package_DIP:DIP-20_W7.62mm_Socket, F.Cu at (227.6, 156.2)
- added LED_BANK1: LED, LED_THT:LED_D5.0mm, F.Cu at (28.6, 271.9)
- added LED_BASIC1: LED, LED_THT:LED_D5.0mm, F.Cu at (28.7, 186.7)
- added LED_DISK1: LED, LED_THT:LED_D5.0mm, F.Cu at (120.6, 125.7)
- added LED_FF1: LED, LED_THT:LED_D5.0mm, F.Cu at (101.8, 287.3)
- added LED_FULL1: LED, LED_THT:LED_D5.0mm, F.Cu at (119.0, 287.4)
- added LED_GFX1: LED, LED_THT:LED_D5.0mm, F.Cu at (28.8, 198.0)
- added LED_HGR1: LED, LED_THT:LED_D5.0mm, F.Cu at (139.8, 287.6)
- added LED_LGR1: LED, LED_THT:LED_D5.0mm, F.Cu at (147.8, 287.6)
- added LED_MIX1: LED, LED_THT:LED_D5.0mm, F.Cu at (127.1, 287.4)
- added LED_PG1: LED, LED_THT:LED_D5.0mm, F.Cu at (28.5, 227.9)
- added LED_PG2: LED, LED_THT:LED_D5.0mm, F.Cu at (28.7, 241.8)
- added LED_RO1: LED, LED_THT:LED_D5.0mm, F.Cu at (69.5, 286.8)
- added LED_RRAM1: LED, LED_THT:LED_D5.0mm, F.Cu at (82.5, 287.1)
- added LED_RROM1: LED, LED_THT:LED_D5.0mm, F.Cu at (90.2, 287.1)
- added LED_RW1: LED, LED_THT:LED_D5.0mm, F.Cu at (61.6, 286.6)
- added LED_TEXT1: LED, LED_THT:LED_D5.0mm, F.Cu at (29.0, 211.3)
- added M1_VID_TXTSHIFT1: SN74LS166AN, Package_DIP:DIP-16_W7.62mm_Socket, F.Cu at (268.2, 123.8)
- added M2_VBUS_LOW1: 74LS245, Package_DIP:DIP-20_W7.62mm_Socket, F.Cu at (197.6, 168.5)
- added M3_VBUS_HIGH1: 74LS245, Package_DIP:DIP-20_W7.62mm_Socket, F.Cu at (197.4, 138.6)
- added M4_ROM_FONTS1: SST39SF040, Package_DIP:DIP-32_W15.24mm_Socket, F.Cu at (245.4, 173.2)
- added N1_SigLatch1: SN74LS279AN, Package_DIP:DIP-16_W7.62mm_Socket, F.Cu at (156.0, 207.7)
- added N2_NOT_SIG1: 74LS14, Package_DIP:DIP-14_W7.62mm_Socket, F.Cu at (135.5, 179.8)
- added N3_ADDR_CNT1: 74LS161, Package_DIP:DIP-16_W7.62mm_Socket, F.Cu at (183.0, 197.3)
- added N4_ADDR_CNT1: 74LS161, Package_DIP:DIP-16_W7.62mm_Socket, F.Cu at (197.8, 198.1)
- added N5_ADDR_CNT1: 74LS161, Package_DIP:DIP-16_W7.62mm_Socket, F.Cu at (213.2, 153.9)
- added N6_ADDR_CNT1: 74LS161, Package_DIP:DIP-16_W7.62mm_Socket, F.Cu at (213.7, 179.8)
- added N7_NOT1: 74LS04, Package_DIP:DIP-14_W7.62mm_Socket, F.Cu at (238.3, 208.8)
- added O1_DECODE_SIGS1: 74LS154, Package_DIP:DIP-24_W15.24mm_Socket, F.Cu at (139.1, 245.0)
- added O2_ROM_VADDR_LOW1: SST39SF040, Package_DIP:DIP-32_W15.24mm_Socket, F.Cu at (213.0, 261.5)
- added O3_ROM_VADDR_HIGH1: SST39SF040, Package_DIP:DIP-32_W15.24mm_Socket, F.Cu at (235.7, 261.7)
- added O4_VidSigLatch1: 74LS574, Package_DIP:DIP-20_W7.62mm_Socket, F.Cu at (219.7, 279.8)
- added P1_Clock1: 25.175MHz, Oscillator:Oscillator_DIP-14, F.Cu at (150.5, 275.2)
- added P2_Clock_Div1: 74LS161, Package_DIP:DIP-16_W7.62mm_Socket, F.Cu at (148.4, 259.8)
- added P3_HORIZ_CNT1: 74LS590, Package_DIP:DIP-16_W7.62mm_Socket, F.Cu at (174.1, 260.2)
- added P4_VERT_CNT1: 74LS590, Package_DIP:DIP-16_W7.62mm_Socket, F.Cu at (174.3, 247.7)
- added P5_VERT_CNT1: 74LS590, Package_DIP:DIP-16_W7.62mm_Socket, F.Cu at (174.2, 234.9)
- added P6_ROM_VGA1: SST39SF040, Package_DIP:DIP-32_W15.24mm_Socket, F.Cu at (211.2, 268.2)
- added Q1: 74LS161, Package_DIP:DIP-16_W7.62mm_Socket, F.Cu at (305.9, 156.6)
- added Q2: 74LS20, Package_DIP:DIP-14_W7.62mm_Socket, F.Cu at (318.2, 158.8)
- added Q3: 4046, Package_DIP:DIP-16_W7.62mm_Socket, F.Cu at (292.5, 156.6)
- added R1: 74LS08, Package_DIP:DIP-14_W7.62mm_Socket, F.Cu at (147.5, 57.6)
- added R10: R, Resistor_SMD:R_0603_1608Metric_Pad0.98x0.95mm_HandSolder, B.Cu at (134.8, 285.2)
- added R11: R, Resistor_SMD:R_0603_1608Metric_Pad0.98x0.95mm_HandSolder, B.Cu at (28.1, 234.1)
- added R12: R, Resistor_SMD:R_0603_1608Metric_Pad0.98x0.95mm_HandSolder, B.Cu at (31.8, 233.9)
- added R13: R, Resistor_SMD:R_0603_1608Metric_Pad0.98x0.95mm_HandSolder, B.Cu at (56.6, 288.7)
- added R14: R, Resistor_SMD:R_0603_1608Metric_Pad0.98x0.95mm_HandSolder, B.Cu at (77.5, 284.2)
- added R15: R, Resistor_SMD:R_0603_1608Metric_Pad0.98x0.95mm_HandSolder, B.Cu at (96.9, 287.7)
- added R16: R, Resistor_SMD:R_0603_1608Metric_Pad0.98x0.95mm_HandSolder, B.Cu at (77.5, 288.7)
- added R17: R, Resistor_SMD:R_0603_1608Metric_Pad0.98x0.95mm_HandSolder, B.Cu at (97.1, 284.2)
- added R18: R, Resistor_SMD:R_0603_1608Metric_Pad0.98x0.95mm_HandSolder, B.Cu at (30.6, 279.0)
- added R19: R, Resistor_SMD:R_0603_1608Metric_Pad0.98x0.95mm_HandSolder, B.Cu at (155.2, 289.3)
- added R2: 74LS245, Package_DIP:DIP-20_W7.62mm_Socket, F.Cu at (134.6, 57.4)
- added R20: R, Resistor_SMD:R_0603_1608Metric_Pad0.98x0.95mm_HandSolder, B.Cu at (134.8, 289.4)
- added R21: R, Resistor_SMD:R_0603_1608Metric_Pad0.98x0.95mm_HandSolder, B.Cu at (29.9, 181.3)
- added R22: R, Resistor_SMD:R_0603_1608Metric_Pad0.98x0.95mm_HandSolder, B.Cu at (119.0, 118.7)
- added R26: 1K, Resistor_SMD:R_0805_2012Metric_Pad1.20x1.40mm_HandSolder, B.Cu at (166.4, 98.4)
- added R27: 1K, Resistor_SMD:R_0805_2012Metric_Pad1.20x1.40mm_HandSolder, B.Cu at (161.1, 85.4)
- added R28: 1K, Resistor_SMD:R_0805_2012Metric_Pad1.20x1.40mm_HandSolder, B.Cu at (204.5, 107.7)
- added R29: 1K, Resistor_SMD:R_0805_2012Metric_Pad1.20x1.40mm_HandSolder, B.Cu at (256.9, 282.6)
- added R3: Pico, MCU_RaspberryPi_and_Boards:RPi_Pico_SMD_TH, F.Cu at (81.9, 69.1)
- added R30: 1K, Resistor_SMD:R_0805_2012Metric_Pad1.20x1.40mm_HandSolder, B.Cu at (256.1, 222.8)
- added R31: 1K, Resistor_SMD:R_0805_2012Metric_Pad1.20x1.40mm_HandSolder, B.Cu at (204.6, 97.2)
- added R34: 30, Resistor_SMD:R_0402_1005Metric_Pad0.72x0.64mm_HandSolder, B.Cu at (296.1, 165.6)
- added R35: R680K, Resistor_SMD:R_0603_1608Metric_Pad0.98x0.95mm_HandSolder, B.Cu at (303.1, 180.8)
- added R36: 51, Resistor_SMD:R_0402_1005Metric_Pad0.72x0.64mm_HandSolder, B.Cu at (298.5, 180.9)
- added R37: 2k2, Resistor_SMD:R_0805_2012Metric_Pad1.20x1.40mm_HandSolder, B.Cu at (306.0, 83.9)
- added R38: 2k2, Resistor_SMD:R_0805_2012Metric_Pad1.20x1.40mm_HandSolder, B.Cu at (312.6, 84.0)
- added R4: 1K, Resistor_SMD:R_0402_1005Metric_Pad0.72x0.64mm_HandSolder, B.Cu at (200.8, 121.7)
- added R41: 1K, Resistor_SMD:R_0402_1005Metric_Pad0.72x0.64mm_HandSolder, B.Cu at (152.3, 193.5)
- added R42: 1K, Resistor_SMD:R_0402_1005Metric_Pad0.72x0.64mm_HandSolder, B.Cu at (156.5, 193.4)
- added R43: 1K, Resistor_SMD:R_0402_1005Metric_Pad0.72x0.64mm_HandSolder, B.Cu at (160.7, 193.7)
- added R5: 1K, Resistor_SMD:R_0402_1005Metric_Pad0.72x0.64mm_HandSolder, B.Cu at (198.3, 129.7)
- added R6: 1K, Resistor_SMD:R_0402_1005Metric_Pad0.72x0.64mm_HandSolder, B.Cu at (193.3, 129.7)
- added R7: R, Resistor_SMD:R_0603_1608Metric_Pad0.98x0.95mm_HandSolder, B.Cu at (28.3, 204.5)
- added R8: R, Resistor_SMD:R_0603_1608Metric_Pad0.98x0.95mm_HandSolder, B.Cu at (32.7, 204.7)
- added R9: R, Resistor_SMD:R_0603_1608Metric_Pad0.98x0.95mm_HandSolder, B.Cu at (114.6, 289.0)
- added RKB1: R, Resistor_SMD:R_0805_2012Metric_Pad1.20x1.40mm_HandSolder, B.Cu at (233.0, 65.1)
- added RKB2: R, Resistor_SMD:R_0805_2012Metric_Pad1.20x1.40mm_HandSolder, B.Cu at (238.0, 65.1)
- added RM1: R, Resistor_SMD:R_0805_2012Metric_Pad1.20x1.40mm_HandSolder, B.Cu at (255.4, 65.1)
- added RM2: R, Resistor_SMD:R_0805_2012Metric_Pad1.20x1.40mm_HandSolder, B.Cu at (260.5, 65.1)
- added R_BLUE_220: 220, Resistor_SMD:R_0603_1608Metric_Pad0.98x0.95mm_HandSolder, B.Cu at (282.0, 74.3)
- added R_BLUE_500: 500, Resistor_SMD:R_0805_2012Metric_Pad1.20x1.40mm_HandSolder, B.Cu at (289.2, 79.3)
- added R_DOWN1: 100, Resistor_SMD:R_0402_1005Metric_Pad0.72x0.64mm_HandSolder, B.Cu at (306.4, 113.7)
- added R_GREEN_220: 220, Resistor_SMD:R_0603_1608Metric_Pad0.98x0.95mm_HandSolder, B.Cu at (271.0, 74.8)
- added R_GREEN_500: 500, Resistor_SMD:R_0805_2012Metric_Pad1.20x1.40mm_HandSolder, B.Cu at (268.7, 79.8)
- added R_POWER1: 330, Resistor_SMD:R_0603_1608Metric_Pad0.98x0.95mm_HandSolder, B.Cu at (41.8, 107.6)
- added R_RED_220: 220, Resistor_SMD:R_0603_1608Metric_Pad0.98x0.95mm_HandSolder, B.Cu at (260.6, 74.3)
- added R_RED_500: 500, Resistor_SMD:R_0805_2012Metric_Pad1.20x1.40mm_HandSolder, B.Cu at (256.6, 78.8)
- added R_RESET_1: 1K, Resistor_SMD:R_0805_2012Metric_Pad1.20x1.40mm_HandSolder, B.Cu at (41.8, 116.5)
- added S1: AY-3-8910, Package_DIP:DIP-40_W15.24mm_Socket, F.Cu at (304.0, 189.6)
- added S2: AY-3-8910, Package_DIP:DIP-40_W15.24mm_Socket, F.Cu at (304.7, 248.9)
- added T1_VIA1: 65C22S, Package_DIP:DIP-40_W15.24mm_Socket, F.Cu at (303.7, 211.0)
- added T2_VIA1: 65C22S, Package_DIP:DIP-40_W15.24mm_Socket, F.Cu at (304.5, 271.3)
- added U1_VID_SHIFT1: ~, Package_DIP:DIP-20_W7.62mm_Socket, F.Cu at (224.8, 124.0)
- added U2_PIXEL_LATCH1: ~, Package_DIP:DIP-20_W7.62mm_Socket, F.Cu at (239.3, 123.8)
- added U3_LOWRES_OUT1: ~, Package_DIP:DIP-20_W7.62mm_Socket, F.Cu at (282.5, 123.3)
- added U4_ODD_BIT1: ~, Package_DIP:DIP-16_W7.62mm_Socket, F.Cu at (253.7, 124.2)
- added V1_PALETTE_LATCH1: ~, Package_DIP:DIP-20_W7.62mm_Socket, F.Cu at (296.4, 123.1)
- added V2_PHI16_LATCH1: ~, Package_DIP:DIP-20_W7.62mm_Socket, F.Cu at (312.4, 123.0)
- added W1: 74LS08, Package_DIP:DIP-14_W7.62mm_Socket, F.Cu at (217.4, 100.9)
- added W2: 74LS04, Package_DIP:DIP-14_W7.62mm_Socket, F.Cu at (231.8, 100.7)
- added W3: 74LS08, Package_DIP:DIP-14_W7.62mm_Socket, F.Cu at (246.8, 100.7)
- added W4: 74LS86, Package_DIP:DIP-14_W7.62mm_Socket, F.Cu at (261.2, 100.6)
- added W5: 74LS08, Package_DIP:DIP-14_W7.62mm_Socket, F.Cu at (275.7, 100.2)
- added W6: 74LS32, Package_DIP:DIP-14_W7.62mm_Socket, F.Cu at (289.5, 100.3)
- added W7: 74LS32, Package_DIP:DIP-14_W7.62mm_Socket, F.Cu at (304.3, 100.6)
- added W8: 74LS32, Package_DIP:DIP-14_W7.62mm_Socket, F.Cu at (318.9, 100.6)
- added Y_MICRO_SD1: Micro_SD_Card, sdcard:microSD_Amazon2, F.Cu at (212.5, 57.4)
- added Y_MICRO_SD2: Micro_SD_Card, sdcard:microSD_Amazon2, F.Cu at (182.2, 57.4)
- added Y_PS2_KB1: PS/2 keyboard, PS2_mini_din_6:MINI-DIN-6-FULL-SHIELD, F.Cu at (236.3, 47.0)
- added Y_PS2_MOUSE1: PS/2 Mouse, PS2_mini_din_6:MINI-DIN-6-FULL-SHIELD, F.Cu at (257.9, 46.9)
- added Y_SERIAL_PINS1: ~, Connector_PinHeader_2.54mm:PinHeader_2x03_P2.54mm_Vertical, F.Cu at (148.7, 81.3)
- added Y_SNES_1: SNES_Controller_Socket, snes:SNES_Controller_Socket, F.Cu at (63.5, 102.6)
- added Y_SNES_2: SNES_Controller_Socket, snes:SNES_Controller_Socket, F.Cu at (111.5, 102.8)
- added Y_VGA1: DB15_Female_HighDensity, Connector_Dsub:DSUB-15-HD_Female_Horizontal_P2.29x1.98mm_EdgePinOffset8.35mm_Housed_MountingHolesOffset10.89mm, F.Cu at (283.1, 61.9)
Other:
- board outline added: 305 x 244 mm
- copper layers 4 -> 2
- board text added: "3RIC 9/28/2024 eric.badger@gmail.com"
