File: kicad/3ric/Communication_sch.kicad_sch (KiCad schematic)
At the start: 16 parts, among them J4_ACIA1 6502-library_65C51N, J5 Conn_02x08_Odd_Even, J6 Conn_02x08_Odd_Even

Commit message: so close!  PCB ready to go?
Connections:
- net GND: now also Y_SERIAL_PINS1.6 (Pin_6)
- net RXD: now also Y_SERIAL_PINS1.3 (Pin_3); no longer Y_SERIAL_PINS1.5 (Pin_5)
- net TXD: now also Y_SERIAL_PINS1.4 (Pin_4); no longer Y_SERIAL_PINS1.6 (Pin_6)
- net VCC: now also Y_SERIAL_PINS1.5 (Pin_5)
- no-connect marks 26 -> 24

Commit message: v2 pcb
Parts:
- removed J5, J6: Conn_02x08_Odd_Even, Connector_PinHeader_2.54mm:PinHeader_2x08_P2.54mm_Vertical, symbol Connector_Generic:Conn_02x08_Odd_Even
- H1_LEVEL_SHIFT1: value ~ -> tsx0108e
- RKB1, RKB2, RM1, RM2: value R -> R1K
Connections:
- net GND: now also J4_ACIA1.16 (~{DCD}), J4_ACIA1.17 (~{DSR})
- no-connect marks 24 -> 22
