File: kicad/3ric/address_decoder.kicad_sch (KiCad schematic)
At the start: 14 parts

Commit message: cleaning up of the schematic
Parts:
- removed B5: 74LS08, symbol 74xx:74LS08
- added unit 3 of A3
- added unit 2 of A3
- added unit 2 of A4
- added unit 3 of A4
- added unit 3 of A5
- added unit 1 of A5
- added unit 2 of A5
- added unit 2 of B1
- added unit 3 of B2
- added unit 4 of B2
- added unit 2 of B5
- added unit 6 of B6
- added unit 5 of B6
- added unit 1 of B6
- added unit 3 of B7
- added unit 1 of B7
- added unit 3 of C2
- added unit 2 of C2
- added unit 5 of C2
- added unit 3 of C5
- added unit 1 of C5
- added unit 2 of C5
- A1, A2, A3, A4, A5, B1, B2, B3, B4, B5, B6, B7, C2, C5: footprint (none) -> Package_DIP:DIP-14_W7.62mm_Socket
Connections:
- net !CA12&!CA13: now also B3.5, B5.1, B5.11
- net !CA13: no longer B5.1
- net !VIDENABLE: now also A5.4
- net PHI2: now also C2.11
- net ~{CS_ROM}: now also A5.5
- new net: A5.1, A5.6
- new net !PHI2: C2.10
- new net C6XX: A5.2
- new net ~{CS_ROM2}: A5.3
- no-connect marks 0 -> 52
Other:
- moved on the sheet: B5A, B5C, B7D

Commit message: pcb layout continued
Connections:
- net B2 renamed BANK2
Other:
- moved on the sheet: A1D
Changed lines of the file:
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@@
 	(wire
 		(pts
-			(xy 119.38 35.56) (xy 121.92 35.56)
+			(xy 120.65 35.56) (xy 121.92 35.56)
 		)
 		(stroke
@@
 	(wire
 		(pts
-			(xy 95.25 33.02) (xy 104.14 33.02)
+			(xy 95.25 33.02) (xy 105.41 33.02)
 		)
 		(stroke
@@
 		)
 	)
-	(global_label "B2"
-		(shape input)
-		(at 104.14 38.1 180)
-		(fields_autoplaced yes)
-		(effects
-			(font
-				(size 1.27 1.27)
-			)
-			(justify right)
-		)
-		(property "Intersheetrefs" "${INTERSHEET_REFS}"
-			(at 99.2474 38.0206 0)
+	(global_label "BANK2"
+		(shape input)
+		(at 105.41 38.1 180)
+		(fields_autoplaced yes)
+		(effects
+			(font
+				(size 1.27 1.27)
+			)
+			(justify right)
+		)
+		(property "Intersheetrefs" "${INTERSHEET_REFS}"
+			(at 96.2562 38.1 0)
 			(effects
 				(font
@@
 	(symbol
 		(lib_id "74xx:74LS08")
-		(at 111.76 35.56 0)
+		(at 113.03 35.56 0)
 		(unit 4)
 		(exclude_from_sim no)
@@
 		(fields_autoplaced yes)
 		(property "Reference" "A1"
-			(at 111.76 28.0502 0)
+			(at 113.03 28.0502 0)
 			(effects
 				(font
@@
 		)
 		(property "Value" "74LS08"
-			(at 111.76 30.5871 0)
+			(at 113.03 30.5871 0)
 			(effects
 				(font
@@
 		)
 		(property "Footprint" "Package_DIP:DIP-14_W7.62mm_Socket"
-			(at 111.76 35.56 0)
+			(at 113.03 35.56 0)
 			(effects
 				(font
@@
 		)
 		(property "Datasheet" "http://www.ti.com/lit/gpn/sn74LS08"
-			(at 111.76 35.56 0)
+			(at 113.03 35.56 0)
 			(effects
 				(font
@@
 		)
 		(property "Description" ""
-			(at 111.76 35.56 0)
-			(effects
-				(font
+			(at 113.03 35.56 0)
+			(effects
+				(font

Commit message: v2 pcb
Parts:
- removed unit 4 of A5
- removed unit 1 of C5
Connections:
- net !CA12&!CA13: no longer B5.1
- net !CA13: now also B5.1
- net !VIDENABLE: now also A4.9; no longer A5.4
- net VIDBUS: now also A5.4
- net ~{CS_RAM}: now also A5.6
- net ~{CS_ROM}: now also A4.10; no longer A5.5
- net ~{RAM}: now also A5.5
- net at A5.1: now also A4.8; no longer A5.6
- no-connect marks 52 -> 46
