File: kicad/3ric/graphicsv2.kicad_sch (KiCad schematic)
At the start: 27 parts

Commit message: pcb layout continued
Connections:
- net !DISPLAY2: now also W2.12
- net DISPLAY2: now reaches W2.13
- no-connect marks 57 -> 55
Other:
- moved on the sheet: W2F
Changed lines of the file:
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@@
 	)
 	(no_connect
-		(at 74.93 229.87)
-	)
-	(no_connect
 		(at 166.37 39.37)
 	)
@@
 	)
 	(no_connect
-		(at 59.69 229.87)
-	)
-	(no_connect
 		(at 25.4 41.91)
 	)
@@
 		)
 	)
+	(global_label "!DISPLAY2"
+		(shape input)
+		(at 46.99 140.97 0)
+		(fields_autoplaced yes)
+		(effects
+			(font
+				(size 1.27 1.27)
+			)
+			(justify left)
+		)
+		(property "Intersheetrefs" "${INTERSHEET_REFS}"
+			(at 59.3491 140.97 0)
+			(effects
+				(font
+					(size 1.27 1.27)
+				)
+				(justify left)
+				(hide yes)
+			)
+		)
+	)
 	(global_label "GND"
 		(shape input)
@@
 		)
 	)
+	(global_label "DISPLAY2"
+		(shape input)
+		(at 31.75 140.97 180)
+		(fields_autoplaced yes)
+		(effects
+			(font
+				(size 1.27 1.27)
+			)
+			(justify right)
+		)
+		(property "Intersheetrefs" "${INTERSHEET_REFS}"
+			(at 19.9957 140.97 0)
+			(effects
+				(font
+					(size 1.27 1.27)
+				)
+				(justify right)
+				(hide yes)
+			)
+		)
+	)
 	(global_label "OddBit2"
 		(shape input)
@@
 	(symbol
 		(lib_id "74xx:74LS04")
-		(at 67.31 229.87 0)
+		(at 39.37 140.97 0)
 		(unit 6)
 		(exclude_from_sim no)
@@
 		(fields_autoplaced yes)
 		(property "Reference" "W2"
-			(at 67.31 222.3602 0)
+			(at 39.37 133.4602 0)
 			(effects
 				(font
@@
 		)
 		(property "Value" "74LS04"
-			(at 67.31 224.8971 0)
+			(at 39.37 135.9971 0)
 			(effects
 				(font
@@
 		)
 		(property "Footprint" "Package_DIP:DIP-14_W7.62mm_Socket"
-			(at 67.31 229.87 0)
+			(at 39.37 140.97 0)
 			(effects
 				(font
@@
 		)
 		(property "Datasheet" "http://www.ti.com/lit/gpn/sn74LS04"
-			(at 67.31 229.87 0)
+			(at 39.37 140.97 0)
 			(effects
 				(font
@@
 		)
 		(property "Description" ""
-			(at 67.31 229.87 0)
+			(at 39.37 140.97 0)
 			(effects
 				(font

Commit message: v2 pcb
Parts:
- R_DOWN1: value 100 -> 1K_0402
- U1_VID_SHIFT1: value ~ -> 74HC299
- U2_PIXEL_LATCH1, U3_LOWRES_OUT1: value ~ -> 74F574
- U4_ODD_BIT1: value ~ -> 74HC161
- V1_PALETTE_LATCH1, V2_PHI16_LATCH1: value ~ -> 74HC574
Connections:
- net VL0: now also U1_VID_SHIFT1.16 (IO7); no longer V1_PALETTE_LATCH1.9 (D7)
- net VL1: now also U1_VID_SHIFT1.4 (IO6); no longer U1_VID_SHIFT1.13 (IO1)
- net VL2: now also U1_VID_SHIFT1.15 (IO5); no longer U1_VID_SHIFT1.6 (IO2)
- net VL3: now also U1_VID_SHIFT1.5 (IO4); no longer U1_VID_SHIFT1.14 (IO3)
- net VL4: now also U1_VID_SHIFT1.14 (IO3); no longer U1_VID_SHIFT1.5 (IO4)
- net VL5: now also U1_VID_SHIFT1.6 (IO2); no longer U1_VID_SHIFT1.15 (IO5)
- net VL6: now also U1_VID_SHIFT1.13 (IO1); no longer U1_VID_SHIFT1.4 (IO6)
- net VL7: now also V1_PALETTE_LATCH1.9 (D7); no longer U1_VID_SHIFT1.16 (IO7)
Changed lines of the file:
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@@
 		)
 	)
-	(global_label "VL0"
+	(global_label "VL7"
 		(shape input)
 		(at 166.37 44.45 180)
@@
 		)
 		(property "Intersheetrefs" "${INTERSHEET_REFS}"
-			(at 160.6307 44.5294 0)
+			(at 160.0586 44.45 0)
 			(effects
 				(font
@@
 		)
 	)
-	(global_label "VL7"
+	(global_label "VL0"
 		(shape input)
 		(at 100.33 52.07 0)
@@
 		)
 		(property "Intersheetrefs" "${INTERSHEET_REFS}"
-			(at 106.0693 52.1494 0)
+			(at 106.6414 52.07 0)
 			(effects
 				(font
@@
 		)
 	)
-	(global_label "VL6"
+	(global_label "VL1"
 		(shape input)
 		(at 100.33 49.53 0)
@@
 		)
 		(property "Intersheetrefs" "${INTERSHEET_REFS}"
-			(at 106.0693 49.6094 0)
+			(at 106.6414 49.53 0)
 			(effects
 				(font
@@
 		)
 	)
-	(global_label "VL2"
+	(global_label "VL5"
 		(shape input)
 		(at 100.33 39.37 0)
@@
 		)
 		(property "Intersheetrefs" "${INTERSHEET_REFS}"
-			(at 106.0693 39.4494 0)
+			(at 106.6414 39.37 0)
 			(effects
 				(font
@@
 		)
 	)
-	(global_label "VL3"
+	(global_label "VL4"
 		(shape input)
 		(at 100.33 41.91 0)
@@
 		)
 		(property "Intersheetrefs" "${INTERSHEET_REFS}"
-			(at 106.0693 41.9894 0)
+			(at 106.6414 41.91 0)
 			(effects
 				(font
@@
 		)
 	)
-	(global_label "VL5"
+	(global_label "VL2"
 		(shape input)
 		(at 100.33 46.99 0)
@@
 		)
 		(property "Intersheetrefs" "${INTERSHEET_REFS}"
-			(at 106.0693 47.0694 0)
+			(at 106.6414 46.99 0)
 			(effects
 				(font
@@
 		)
 	)
-	(global_label "VL1"
+	(global_label "VL6"
 		(shape input)
 		(at 100.33 36.83 0)
@@
 		)
 		(property "Intersheetrefs" "${INTERSHEET_REFS}"
-			(at 106.0693 36.9094 0)
+			(at 106.6414 36.83 0)
 			(effects
 				(font
@@
 		)
 	)
-	(global_label "VL4"
+	(global_label "VL3"
 		(shape input)
 		(at 100.33 44.45 0)
@@
 		)
 		(property "Intersheetrefs" "${INTERSHEET_REFS}"
-			(at 106.0693 44.5294 0)
+			(at 106.6414 44.45 0)
 			(effects
 				(font
@@
 			)
 		)
-		(property "Value" "~"
+		(property "Value" "74HC161"
 			(at 263.6394 22.9671 0)
 			(effects
@@
 			)
 		)
-		(property "Value" "~"
+		(property "Value" "74F574"
 			(at 222.9994 22.9671 0)
 			(effects
@@
 			)
 		)
-		(property "Value" "~"
+		(property "Value" "74HC574"
 			(at 40.1194 25.5071 0)
 			(effects
@@
 			)
 		)
-		(property "Value" "~"
+		(property "Value" "74HC574"
 			(at 181.0894 22.9671 0)
 			(effects
@@
 			)
 		)
-		(property "Value" "~"
+		(property "Value" "74HC299"
 			(at 89.6494 22.9671 0)
 			(effects
@@
 			)
 		)
-		(property "Value" "100"
+		(property "Value" "1K_0402"
 			(at 227.33 81.6411 90)
 			(effects
@@
 			)
 		)
-		(property "Value" "~"
+		(property "Value" "74F574"
 			(at 135.3694 22.9671 0)
 			(effects
