File: kicad/3ric/romdisk_sch.kicad_sch (KiCad schematic)
At the start: 4 parts, among them J2 Conn_02x03_Odd_Even

Commit message: so close!  PCB ready to go?
Connections:
- net ROM2: now also J2.5 (Pin_5); no longer J2.3 (Pin_3)
- net ROM3: now also J2.3 (Pin_3); no longer J2.5 (Pin_5)
Changed lines of the file:
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@@
 	(global_label "ROM2"
+		(shape input)
+		(at 66.04 148.59 180)
+		(fields_autoplaced yes)
+		(effects
+			(font
+				(size 1.27 1.27)
+			)
+			(justify right)
+		)
+		(property "Intersheetrefs" "${INTERSHEET_REFS}"
+			(at 57.7934 148.59 0)
+			(effects
+				(font
+					(size 1.27 1.27)
+				)
+				(justify right)
+				(hide yes)
+			)
+		)
+	)
+	(global_label "ROM3"
 		(shape input)
 		(at 66.04 146.05 180)
@@
 			(effects
 				(font
-					(size 1.27 1.27)
-				)
-				(justify right)
-				(hide yes)
-			)
-		)
-	)
-	(global_label "ROM3"
-		(shape input)
-		(at 66.04 148.59 180)
-		(fields_autoplaced yes)
-		(effects
-			(font
-				(size 1.27 1.27)
-			)
-			(justify right)
-		)
-		(property "Intersheetrefs" "${INTERSHEET_REFS}"
-			(at 57.7934 148.59 0)
-			(effects
-				(font

Commit message: v2 pcb
Parts:
- R41, R42, R43: value 1K -> 1K_0402
Changed lines of the file:
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@@
 			)
 		)
-		(property "Value" "1K"
+		(property "Value" "1K_0402"
 			(at 107.95 140.5636 90)
 			(effects
@@
 			)
 		)
-		(property "Value" "1K"
+		(property "Value" "1K_0402"
 			(at 107.95 132.9436 90)
 			(effects
@@
 			)
 		)
-		(property "Value" "1K"
+		(property "Value" "1K_0402"
 			(at 107.95 148.1836 90)
 			(effects
