File: kicad/3ric/vg_memsignal.kicad_sch (KiCad schematic)
At the start: 3 parts

Commit message: v2 pcb
Other:
- note removed: "todo: update from breadboard"
Changed lines of the file:
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@@
-		)
-	)
-	(text "todo: update from breadboard\n"
-		(exclude_from_sim no)
-		(at 67.31 90.17 0)
-		(effects
-			(font
-				(size 1.27 1.27)
-			)
-			(justify left bottom)
 		)
 	)
