File: kicad/3ric/vgatiming.kicad_sch (KiCad schematic)
At the start: 7 parts, among them P1_Clock 25.175MHz, P2_Clock_Div 74LS161, P3_HORIZ_CNT 74LS590, P4_VERT_CNT 74LS590, P5_VERT_CNT 74LS590, P6_ROM_VGA SST39SF040

Commit message: cleaning up of the schematic
Parts:
- renumbered O4_VidSigLatch to O4_VidSigLatch1, P1_Clock to P1_Clock1, P2_Clock_Div to P2_Clock_Div1, P3_HORIZ_CNT to P3_HORIZ_CNT1, P4_VERT_CNT to P4_VERT_CNT1, P5_VERT_CNT to P5_VERT_CNT1, P6_ROM_VGA to P6_ROM_VGA1
Connections:
- net PHI4: now also P2_Clock_Div1.12 (Q2), P3_HORIZ_CNT1.13 (CPR)
- net DISPLAY4: no longer names the net of O4_VidSigLatch1.12 (Q7)
- no-connect marks 14 -> 15
Changed lines of the file:
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@@
 	(paper "A4")
+	(junction
+		(at 115.57 71.12)
+		(diameter 0)
+		(color 0 0 0 0)
+	)
 	(junction
 		(at 55.88 106.68)
@@
 	)
 	(no_connect
+		(at 265.43 91.44)
+	)
+	(no_connect
 		(at 156.21 55.88)
 	)
@@
 	(wire
 		(pts
-			(xy 115.57 48.26) (xy 115.57 99.06)
+			(xy 115.57 48.26) (xy 115.57 71.12)
 		)
 		(stroke
@@
 	(wire
 		(pts
-			(xy 134.62 53.34) (xy 135.89 53.34)
+			(xy 115.57 71.12) (xy 115.57 99.06)
 		)
 		(stroke
@@
 	(wire
 		(pts
-			(xy 55.88 91.44) (xy 55.88 106.68)
+			(xy 134.62 53.34) (xy 135.89 53.34)
 		)
 		(stroke
@@
 	(wire
 		(pts
-			(xy 115.57 48.26) (xy 135.89 48.26)
+			(xy 55.88 91.44) (xy 55.88 106.68)
 		)
 		(stroke
@@
 	(wire
 		(pts
-			(xy 128.27 146.05) (xy 135.89 146.05)
+			(xy 115.57 48.26) (xy 135.89 48.26)
 		)
 		(stroke
@@
 	(wire
 		(pts
-			(xy 156.21 114.3) (xy 158.75 114.3)
+			(xy 113.03 71.12) (xy 115.57 71.12)
 		)
 		(stroke
@@
 	(wire
 		(pts
-			(xy 55.88 106.68) (xy 59.69 106.68)
+			(xy 128.27 146.05) (xy 135.89 146.05)
 		)
 		(stroke
@@
 	(wire
 		(pts
-			(xy 158.75 114.3) (xy 158.75 128.27)
+			(xy 156.21 114.3) (xy 158.75 114.3)
 		)
 		(stroke
@@
 	(wire
 		(pts
-			(xy 240.03 81.28) (xy 222.25 81.28)
+			(xy 55.88 106.68) (xy 59.69 106.68)
 		)
 		(stroke
@@
 		)
 	)
+	(wire
+		(pts
+			(xy 158.75 114.3) (xy 158.75 128.27)
+		)
+		(stroke
+			(width 0)
+			(type default)
+		)
+	)
+	(wire
+		(pts
+			(xy 240.03 81.28) (xy 222.25 81.28)
+		)
+		(stroke
+			(width 0)
+			(type default)
+		)
+	)
 	(global_label "VCC"
 		(shape input)
@@
 		)
 	)
+	(global_label "PHI4"
+		(shape input)
+		(at 113.03 71.12 180)
+		(fields_autoplaced yes)
+		(effects
+			(font
+				(size 1.27 1.27)
+			)
+			(justify right)
+		)
+		(property "Intersheetrefs" "${INTERSHEET_REFS}"
+			(at 105.63 71.12 0)
+			(effects
+				(font
+					(size 1.27 1.27)
+				)
+				(justify right)
+				(hide yes)
+			)
+		)
+	)
 	(global_label "GND"
 		(shape input)
@@
 				)
 				(justify right)
-				(hide yes)
-			)
-		)
-	)
-	(global_label "DISPLAY4"
-		(shape input)
-		(at 265.43 91.44 0)
-		(fields_autoplaced yes)
-		(effects
-			(font
-				(size 1.27 1.27)
-			)
-			(justify left)
-		)
-		(property "Intersheetrefs" "${INTERSHEET_REFS}"
-			(at 276.6121 91.3606 0)
-			(effects
-				(font
-					(size 1.27 1.27)
-				)
-				(justify left)
 				(hide yes)
 			)
@@
 		(dnp no)
 		(fields_autoplaced yes)
-		(property "Reference" "P5_VERT_CNT"
+		(property "Reference" "P5_VERT_CNT1"
 			(at 148.0694 134.7302 0)
 			(effects
@@
 			(project "3ric"
 				(path "/e63e39d7-6ac0-4ffd-8aa3-1841a4541b55/16ecb62b-433c-4b3d-ae08-a168010e2dc7"
-					(reference "P5_VERT_CNT")
+					(reference "P5_VERT_CNT1")
 					(unit 1)
 				)
@@
 		(dnp no)
 		(fields_autoplaced yes)
-		(property "Reference" "O4_VidSigLatch"
+		(property "Reference" "O4_VidSigLatch1"
 			(at 254.7494 67.4202 0)
 			(effects
@@
 			(project "3ric"
 				(path "/e63e39d7-6ac0-4ffd-8aa3-1841a4541b55/16ecb62b-433c-4b3d-ae08-a168010e2dc7"
-					(reference "O4_VidSigLatch")
+					(reference "O4_VidSigLatch1")
 					(unit 1)
 				)
@@
 		(dnp no)
 		(fields_autoplaced yes)
-		(property "Reference" "P3_HORIZ_CNT"
+		(property "Reference" "P3_HORIZ_CNT1"
 			(at 148.0694 34.4002 0)
 			(effects
@@
 			(project "3ric"
 				(path "/e63e39d7-6ac0-4ffd-8aa3-1841a4541b55/16ecb62b-433c-4b3d-ae08-a168010e2dc7"
-					(reference "P3_HORIZ_CNT")
+					(reference "P3_HORIZ_CNT1")
 					(unit 1)
 				)
@@
 		(dnp no)
 		(fields_autoplaced yes)
-		(property "Reference" "P4_VERT_CNT"
+		(property "Reference" "P4_VERT_CNT1"
 			(at 148.0694 85.2002 0)
 			(effects
@@
 			(project "3ric"
 				(path "/e63e39d7-6ac0-4ffd-8aa3-1841a4541b55/16ecb62b-433c-4b3d-ae08-a168010e2dc7"
-					(reference "P4_VERT_CNT")
+					(reference "P4_VERT_CNT1")
 					(unit 1)
 				)
@@
 		(dnp no)
 		(fields_autoplaced yes)
-		(property "Reference" "P2_Clock_Div"
+		(property "Reference" "P2_Clock_Div1"
 			(at 85.8394 87.7402 0)
 			(effects
@@
 			(project "3ric"
 				(path "/e63e39d7-6ac0-4ffd-8aa3-1841a4541b55/16ecb62b-433c-4b3d-ae08-a168010e2dc7"
-					(reference "P2_Clock_Div")
+					(reference "P2_Clock_Div1")
 					(unit 1)
 				)
@@
 		(on_board yes)
 		(dnp no)
-		(property "Reference" "P6_ROM_VGA"
+		(property "Reference" "P6_ROM_VGA1"
 			(at 207.01 66.5226 0)
 			(effects
@@
 			(project "3ric"
 				(path "/e63e39d7-6ac0-4ffd-8aa3-1841a4541b55/16ecb62b-433c-4b3d-ae08-a168010e2dc7"
-					(reference "P6_ROM_VGA")
+					(reference "P6_ROM_VGA1")
 					(unit 1)
 				)
@@
 		(on_board yes)
 		(dnp no)
-		(property "Reference" "P1_Clock"
+		(property "Reference" "P1_Clock1"
 			(at 34.4424 105.5116 0)
 			(effects
@@
 			(project "3ric"
 				(path "/e63e39d7-6ac0-4ffd-8aa3-1841a4541b55/16ecb62b-433c-4b3d-ae08-a168010e2dc7"
-					(reference "P1_Clock")
+					(reference "P1_Clock1")
 					(unit 1)
 				)

Commit message: v2 pcb
Parts:
- added C13: C60, Capacitor_SMD:C_0805_2012Metric_Pad1.18x1.45mm_HandSolder, symbol Device:C
Connections:
- net PHI16: now also C13.1
- net PHI8: now also C13.2
Changed lines of the file:
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@@
+	(wire
+		(pts
+			(xy 105.41 96.52) (xy 96.52 96.52)
+		)
+		(stroke
+			(width 0)
+			(type default)
+		)
+	)
 	(wire
 		(pts
@@
 	(wire
 		(pts
+			(xy 105.41 93.98) (xy 96.52 93.98)
+		)
+		(stroke
+			(width 0)
+			(type default)
+		)
+	)
+	(wire
+		(pts
 			(xy 240.03 83.82) (xy 222.25 83.82)
 		)
@@
 		)
 	)
+	(global_label "PHI16"
+		(shape input)
+		(at 83.82 66.04 180)
+		(fields_autoplaced yes)
+		(effects
+			(font
+				(size 1.27 1.27)
+			)
+			(justify right)
+		)
+		(property "Intersheetrefs" "${INTERSHEET_REFS}"
+			(at 75.2105 66.04 0)
+			(effects
+				(font
+					(size 1.27 1.27)
+				)
+				(justify right)
+				(hide yes)
+			)
+		)
+	)
 	(global_label "DISPLAY3"
 		(shape input)
@@
 		)
 	)
+	(global_label "PHI8"
+		(shape input)
+		(at 83.82 73.66 180)
+		(fields_autoplaced yes)
+		(effects
+			(font
+				(size 1.27 1.27)
+			)
+			(justify right)
+		)
+		(property "Intersheetrefs" "${INTERSHEET_REFS}"
+			(at 76.42 73.66 0)
+			(effects
+				(font
+					(size 1.27 1.27)
+				)
+				(justify right)
+				(hide yes)
+			)
+		)
+	)
 	(global_label "GND"
 		(shape input)
@@
 	(global_label "PHI16"
 		(shape input)
-		(at 96.52 93.98 0)
-		(fields_autoplaced yes)
-		(effects
-			(font
-				(size 1.27 1.27)
-			)
-			(justify left)
-		)
-		(property "Intersheetrefs" "${INTERSHEET_REFS}"
-			(at 104.5574 93.9006 0)
+		(at 105.41 93.98 0)
+		(fields_autoplaced yes)
+		(effects
+			(font
+				(size 1.27 1.27)
+			)
+			(justify left)
+		)
+		(property "Intersheetrefs" "${INTERSHEET_REFS}"
+			(at 113.4474 93.9006 0)
 			(effects
 				(font
@@
 	(global_label "PHI8"
 		(shape input)
-		(at 96.52 96.52 0)
-		(fields_autoplaced yes)
-		(effects
-			(font
-				(size 1.27 1.27)
-			)
-			(justify left)
-		)
-		(property "Intersheetrefs" "${INTERSHEET_REFS}"
-			(at 103.3479 96.4406 0)
+		(at 105.41 96.52 0)
+		(fields_autoplaced yes)
+		(effects
+			(font
+				(size 1.27 1.27)
+			)
+			(justify left)
+		)
+		(property "Intersheetrefs" "${INTERSHEET_REFS}"
+			(at 112.2379 96.4406 0)
 			(effects
 				(font
@@
 					(unit 1)
 				)
+			)
+		)
+	)
+	(symbol
+		(lib_id "Device:C")
+		(at 83.82 69.85 0)
+		(unit 1)
+		(exclude_from_sim no)
+		(in_bom yes)
+		(on_board yes)
+		(dnp no)
+		(property "Reference" "C13"
+			(at 86.868 68.58 0)
+			(effects
+				(font
+					(size 1.27 1.27)
+				)
+				(justify left)
+			)
+		)
+		(property "Value" "C60"
+			(at 86.614 70.866 0)
+			(effects
+				(font
+					(size 1.27 1.27)
+				)
+				(justify left)
+			)
+		)
+		(property "Footprint" "Capacitor_SMD:C_0805_2012Metric_Pad1.18x1.45mm_HandSolder"
+			(at 84.7852 73.66 0)
+			(effects
+				(font
+					(size 1.27 1.27)
+				)
+				(hide yes)
+			)
+		)
+		(property "Datasheet" "~"
+			(at 83.82 69.85 0)
+			(effects
+				(font
+					(size 1.27 1.27)
+				)
+				(hide yes)
+			)
+		)
+		(property "Description" ""
+			(at 83.82 69.85 0)
+			(effects
+				(font
+					(size 1.27 1.27)
+				)
+				(hide yes)
+			)
+		)
+		(pin "1"
+		)
+		(pin "2"
+		)
+		(instances
+			(project "3ric"
+				(path "/e63e39d7-6ac0-4ffd-8aa3-1841a4541b55/16ecb62b-433c-4b3d-ae08-a168010e2dc7"
+					(reference "C13")
+					(unit 1)
+				)
